File: purple_pill.sch (KiCad schematic (older format))
At the start: 17 parts, among them CN1 Conn_01x28_MountingPin, CN2 Conn_01x28_MountingPin, U1 STM32F405RGTx

Commit message: Oscilators and Power
Parts:
- added C? (x2): 20pF, symbol Device:C
- added C? (x2): 12.5pF, symbol Device:C
- added C? (x4): 100nF, symbol Device:C
- added X1: 8Mhz, Crystal:Crystal_SMD_Abracon_ABM8G-4Pin_3.2x2.5mm, symbol Device:Crystal_GND24_Small
- added X2: 32.768KHz, Crystal:Crystal_SMD_3215-2Pin_3.2x1.5mm, symbol Device:Crystal
- J?: symbol Connector:Conn_ARM_JTAG_SWD_10 -> purple_pill-rescue:Conn_ARM_JTAG_SWD_10-Connector
Connections:
- net labels removed: OSC32IN, OSC32OUT, OSCIN, OSCOUT
- wire segments 78 -> 114

Commit message: Schmeatic Complete - Maybe...
Parts:
- removed CN1, CN2: Conn_01x28_MountingPin, symbol Connector_Generic_MountingPin:Conn_01x28_MountingPin
- added C? (x2): 2.2uF, Capacitor_SMD:C_0805_2012Metric_Pad1.15x1.40mm_HandSolder, symbol Device:C
- added J1, J2: Conn_01x24_MountingPin, Connector_PinHeader_2.54mm:PinHeader_1x24_P2.54mm_Vertical, symbol Connector_Generic_MountingPin:Conn_01x24_MountingPin
- added JP? (x5): Jumper_NC_Small, Jumper:SolderJumper-2_P1.3mm_Open_TrianglePad1.0x1.5mm, symbol Device:Jumper_NC_Small
- added JP?: Jumper_3_Bridged12, Jumper:SolderJumper-3_P2.0mm_Open_TrianglePad1.0x1.5mm_NumberLabels, symbol Jumper:Jumper_3_Bridged12
- C? (x10): footprint (none) -> Capacitor_SMD:C_0805_2012Metric_Pad1.15x1.40mm_HandSolder
- J?: footprint (none) -> Connector_USB:USB_C_Receptacle_Amphenol_12401610E4-2A
- R? (x8): footprint (none) -> Resistor_SMD:R_0805_2012Metric_Pad1.15x1.40mm_HandSolder
- R?: footprint Resistor_SMD:R_0805_2012Metric -> Resistor_SMD:R_0805_2012Metric_Pad1.15x1.40mm_HandSolder
Connections:
- net labels added: GNDA
- wire segments 114 -> 234
- no-connect marks 3 -> 4

Commit message: Initial Board Layout
Parts:
- gave numbers to parts that had none: 30

Commit message: PCB Layout Complete
 On branch master
 Changes to be committed:
	modified:   purple_pill.kicad_pcb
	modified:   purple_pill.pro
	modified:   purple_pill.sch
Parts:
- removed C10, C12: 100nF, Capacitor_SMD:C_0805_2012Metric_Pad1.15x1.40mm_HandSolder, symbol Device:C
- removed JP5: Jumper_NC_Small, Jumper:SolderJumper-2_P1.3mm_Open_TrianglePad1.0x1.5mm, symbol Device:Jumper_NC_Small
Connections:
- net labels removed: GNDA
- wire segments 234 -> 227
- no-connect marks 4 -> 6
Changed lines of the file:
@@
 EESchema Schematic File Version 4
 LIBS:purple_pill-cache
-EELAYER 29 0
+EELAYER 26 0
 EELAYER END
 $Descr A 11000 8500
@@
 	1    0    0    -1
 $EndComp
-$Comp
-L Device:C C10
-U 1 1 5CE0D791
-P 7250 5950
-F 0 "C10" H 7365 5996 50  0000 L CNN
-F 1 "100nF" H 7365 5905 50  0000 L CNN
-F 2 "Capacitor_SMD:C_0805_2012Metric_Pad1.15x1.40mm_HandSolder" H 7288 5800 50  0001 C CNN
-F 3 "~" H 7250 5950 50  0001 C CNN
-	1    7250 5950
-	1    0    0    -1
-$EndComp
-$Comp
-L Device:C C12
-U 1 1 5CE0DD28
-P 7750 5950
-F 0 "C12" H 7865 5996 50  0000 L CNN
-F 1 "100nF" H 7865 5905 50  0000 L CNN
-F 2 "Capacitor_SMD:C_0805_2012Metric_Pad1.15x1.40mm_HandSolder" H 7788 5800 50  0001 C CNN
-F 3 "~" H 7750 5950 50  0001 C CNN
-	1    7750 5950
-	1    0    0    -1
-$EndComp
 Wire Wire Line
 	6250 5550 6250 5800
@@
 	6250 5800 6750 5800
 Connection ~ 6250 5800
-Connection ~ 6750 5800
-Wire Wire Line
-	6750 5800 7250 5800
-Connection ~ 7250 5800
-Wire Wire Line
-	7250 5800 7750 5800
-Wire Wire Line
-	7750 6100 7250 6100
-Connection ~ 6750 6100
 Wire Wire Line
 	6750 6100 6250 6100
-Connection ~ 7250 6100
-Wire Wire Line
-	7250 6100 6750 6100
 Wire Wire Line
 	6250 6100 6250 6350
@@
 L power:GND #PWR0114
 U 1 1 5D325A4C
-P 5100 5500
-F 0 "#PWR0114" H 5100 5250 50  0001 C CNN
-F 1 "GND" H 5105 5327 50  0000 C CNN
-F 2 "" H 5100 5500 50  0001 C CNN
-F 3 "" H 5100 5500 50  0001 C CNN
-	1    5100 5500
-	1    0    0    -1
-$EndComp
-Wire Wire Line
-	5100 5350 5100 5500
-$Comp
-L power:GNDA #PWR0115
-U 1 1 5D3359AF
-P 5300 5500
-F 0 "#PWR0115" H 5300 5250 50  0001 C CNN
-F 1 "GNDA" H 5305 5327 50  0000 C CNN
-F 2 "" H 5300 5500 50  0001 C CNN
-F 3 "" H 5300 5500 50  0001 C CNN
-	1    5300 5500
-	1    0    0    -1
-$EndComp
-$Comp
-L power:GNDA #PWR0116
-U 1 1 5D34C82E
-P 950 4350
-F 0 "#PWR0116" H 950 4100 50  0001 C CNN
-F 1 "GNDA" H 955 4177 50  0000 C CNN
-F 2 "" H 950 4350 50  0001 C CNN
-F 3 "" H 950 4350 50  0001 C CNN
-	1    950  4350
-	1    0    0    -1
-$EndComp
-Wire Wire Line
-	1300 4250 950  4250
-Wire Wire Line
-	950  4250 950  4350
-$Comp
-L power:GNDA #PWR0117
-U 1 1 5D35CDB4
-P 950 7300
-F 0 "#PWR0117" H 950 7050 50  0001 C CNN
-F 1 "GNDA" H 955 7127 50  0000 C CNN
-F 2 "" H 950 7300 50  0001 C CNN
-F 3 "" H 950 7300 50  0001 C CNN
-	1    950  7300
-	1    0    0    -1
-$EndComp
-Wire Wire Line
-	1300 7200 950  7200
-Wire Wire Line
-	950  7200 950  7300
+P 5200 5050
+F 0 "#PWR0114" H 5200 4800 50  0001 C CNN
+F 1 "GND" H 5205 4877 50  0000 C CNN
+F 2 "" H 5200 5050 50  0001 C CNN
+F 3 "" H 5200 5050 50  0001 C CNN
+	1    5200 5050
+	1    0    0    -1
+$EndComp
 $Comp
 L power:+3V3 #PWR0118
@@
 	5100 850  5100 1050
 $Comp
-L Device:Jumper_NC_Small JP5
-U 1 1 5D3D41E6
-P 5200 5350
-F 0 "JP5" H 5200 5562 50  0000 C CNN
-F 1 "Jumper_NC_Small" H 5200 5471 50  0000 C CNN
-F 2 "Jumper:SolderJumper-2_P1.3mm_Open_TrianglePad1.0x1.5mm" H 5200 5350 50  0001 C CNN
-F 3 "~" H 5200 5350 50  0001 C CNN
-	1    5200 5350
-	1    0    0    -1
-$EndComp
-Wire Wire Line
-	5300 5500 5300 5350
-Connection ~ 5300 5350
-Connection ~ 5100 5350
-$Comp
 L power:GND #PWR0119
 U 1 1 5D3F70C5
@@
 	0    1    1    0
 $EndComp
-Wire Wire Line
-	5300 4750 5300 5350
-Wire Wire Line
-	5100 4850 5100 5350
-Connection ~ 5100 4850
 $Comp
 L Jumper:Jumper_3_Bridged12 JP3
@@
 Wire Wire Line
 	7900 3800 7800 3800
+Wire Wire Line
+	5300 4750 5300 4850
+Wire Wire Line
+	5300 4850 5200 4850
+Connection ~ 5200 4850
+Wire Wire Line
+	5200 4850 5200 5050
+Wire Wire Line
+	1300 4250 1300 4350
+Connection ~ 1300 4350
+Wire Wire Line
+	1300 7200 1300 7300
+Connection ~ 1300 7300
+NoConn ~ 1500 4550
+NoConn ~ 1500 7500
 $EndSCHEMATC
